Commit message: feat: adding debugging dashboard

File: seaweed_description/urdf/diff_thrust_wamv/wamv_target.urdf (robot description, URDF)
Before this commit: robot WAM-V, 24 links, 23 joints
Links:
- removed link wamv/back_left_engine_link
- removed link wamv/back_left_propeller_link
- removed link wamv/back_right_engine_link
- removed link wamv/back_right_propeller_link
- removed link wamv/ball_shooter_base_link
- removed link wamv/ball_shooter_launcher_link
- removed link wamv/base_link
- removed link wamv/camera_link
- removed link wamv/camera_link_optical
- removed link wamv/camera_post_arm_link
- removed link wamv/camera_post_link
- removed link wamv/cpu_cases_link
- removed link wamv/front_left_engine_link
- removed link wamv/front_left_propeller_link
- removed link wamv/front_right_engine_link
- removed link wamv/front_right_propeller_link
- removed link wamv/gps_wamv_link
- removed link wamv/imu_wamv_link
- removed link wamv/left_battery_link
- removed link wamv/lidar_wamv_link
- removed link wamv/lidar_wamv_post_arm_link
- removed link wamv/lidar_wamv_post_link
- removed link wamv/receiver
- removed link wamv/right_battery_link
- added link back_left_engine_link, mass 15; collision box size=0.12 0.15 0.12; collision box size=0.2 0.15 0.83
- added link back_left_propeller_link, mass 0.5; collision cylinder length=0.18 radius=0.24; visual mesh filename=package://wamv_description/models/propeller/mesh/propeller.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
- added link back_right_engine_link, mass 15; collision box size=0.12 0.15 0.12; collision box size=0.2 0.15 0.83
- added link back_right_propeller_link, mass 0.5; collision cylinder length=0.18 radius=0.24; visual mesh filename=package://wamv_description/models/propeller/mesh/propeller.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
- added link ball_shooter_base_link, mass 0.5; visual mesh filename=package://vrx_gazebo/models/ball_shooter/meshes/ball_shoote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
- added link ball_shooter_launcher_link, mass 0.5; collision box size=0.3 0.3 0.2; visual mesh filename=package://vrx_gazebo/models/ball_shooter/meshes/ball_shoote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
- added link base_link, mass 180.0; collision box size=0.65 0.2 0.1; collision box size=0.65 0.2 0.1
- added link camera_link, mass 0.3; collision box size=0.036 0.03 0.03; collision cylinder length=0.042 radius=0.015
- added link camera_link_optical
- added link camera_post_arm_link, mass 0.1; collision cylinder length=0.065 radius=0.008; visual mesh filename=package://vrx_gazebo/models/sensor_post/mesh/sensor_post_ar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
- added link camera_post_link, mass 0.15885000000000002; collision cylinder length=0.17650000000000002 radius=0.0076; visual cylinder length=0.17650000000000002 radius=0.0076
- added link cpu_cases_link, mass 20; collision box size=0.375 0.64 0.28; collision box size=0.595 0.83 0.47
- added link front_left_engine_link, mass 15; collision box size=0.12 0.15 0.12; collision box size=0.2 0.15 0.83
- added link front_left_propeller_link, mass 0.5; collision cylinder length=0.18 radius=0.24; visual mesh filename=package://wamv_description/models/propeller/mesh/propeller.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
- added link front_right_engine_link, mass 15; collision box size=0.12 0.15 0.12; collision box size=0.2 0.15 0.83
- added link front_right_propeller_link, mass 0.5; collision cylinder length=0.18 radius=0.24; visual mesh filename=package://wamv_description/models/propeller/mesh/propeller.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
- added link gps_wamv_link, mass 1; collision cylinder length=0.05 radius=0.015; collision cylinder length=0.1 radius=0.15
- added link imu_wamv_link, mass 0.1; collision box size=0.05 0.025 0.005; visual box size=0.05 0.025 0.005
- added link left_battery_link, mass 23.5; collision box size=.6 .4 .31; visual mesh filename=package://vrx_gazebo/models/battery/mesh/battery.dae
- added link lidar_wamv_link, mass 1; collision cylinder length=0.075 radius=0.055; visual mesh filename=package://vrx_gazebo/models/3d_lidar/mesh/3d_lidar.dae
- added link lidar_wamv_post_arm_link, mass 0.1; collision cylinder length=0.065 radius=0.008; visual mesh filename=package://vrx_gazebo/models/sensor_post/mesh/sensor_post_ar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
- added link lidar_wamv_post_link, mass 0.40815000000000007; collision cylinder length=0.45350000000000007 radius=0.0076; visual cylinder length=0.45350000000000007 radius=0.0076
- added link receiver, mass 0.1; visual sphere radius=0.01
- added link right_battery_link, mass 23.5; collision box size=.6 .4 .31; visual mesh filename=package://vrx_gazebo/models/battery/mesh/battery.dae
Joints:
- removed joint wamv/back_left_chassis_engine_joint
- removed joint wamv/back_left_engine_propeller_joint
- removed joint wamv/back_right_chassis_engine_joint
- removed joint wamv/back_right_engine_propeller_joint
- removed joint wamv/ball_shooter_base_joint
- removed joint wamv/ball_shooter_launcher_joint
- removed joint wamv/base_to_camera_post_joint
- removed joint wamv/base_to_lidar_wamv_post_joint
- removed joint wamv/camera_post_arm_to_camera_joint
- removed joint wamv/camera_post_to_camera_post_arm_joint
- removed joint wamv/camera_to_camera_link_optical_joint
- removed joint wamv/chasis_cpu_cases_joint
- removed joint wamv/front_left_chassis_engine_joint
- removed joint wamv/front_left_engine_propeller_joint
- removed joint wamv/front_right_chassis_engine_joint
- removed joint wamv/front_right_engine_propeller_joint
- removed joint wamv/gps_wamv_joint
- removed joint wamv/imu_wamv_joint
- removed joint wamv/left_chasis_battery_joint
- removed joint wamv/lidar_wamv_post_arm_to_lidar_wamv_joint
- removed joint wamv/lidar_wamv_post_to_lidar_wamv_post_arm_joint
- removed joint wamv/receiver_pinger_joint
- removed joint wamv/right_chasis_battery_joint
- added joint back_left_chassis_engine_joint: type revolute, parent base_link, child back_left_engine_link, origin xyz=-2.4 1 0 rpy=0.0 0.0 0, axis 0 0 1, limit lower=-3.141592653589793 upper=3.141592653589793 effort=10 velocity=10
- added joint back_left_engine_propeller_joint: type continuous, parent back_left_engine_link, child back_left_propeller_link, origin xyz=-0.278156 0 -0.509371 rpy=0 0 0, axis 1 0 0, limit effort=100 velocity=100
- added joint back_right_chassis_engine_joint: type revolute, parent base_link, child back_right_engine_link, origin xyz=-2.4 -1 0 rpy=0.0 0.0 0, axis 0 0 1, limit lower=-3.141592653589793 upper=3.141592653589793 effort=10 velocity=10
- added joint back_right_engine_propeller_joint: type continuous, parent back_right_engine_link, child back_right_propeller_link, origin xyz=-0.278156 0 -0.509371 rpy=0 0 0, axis 1 0 0, limit effort=100 velocity=100
- added joint ball_shooter_base_joint: type revolute, parent base_link, child ball_shooter_base_link, origin xyz=0.55 -0.3 1.3 rpy=0 0 0.0, axis 0 0 1, limit lower=0.0 upper=0 effort=1000.0 velocity=0
- added joint ball_shooter_launcher_joint: type revolute, parent ball_shooter_base_link, child ball_shooter_launcher_link, origin xyz=-0.0204 0 0.107877 rpy=0 -0.3490658503988659 0, axis 0 0 1, limit lower=0.0 upper=0 effort=1000.0 velocity=0
- added joint base_to_camera_post_joint: type fixed, parent base_link, child camera_post_link, origin xyz=0.7 0.0 1.38475 rpy=0 0 0.0
- added joint base_to_lidar_wamv_post_joint: type fixed, parent base_link, child lidar_wamv_post_link, origin xyz=0.6299999999999999 0.0 1.52325 rpy=0 0 0.0
- added joint camera_post_arm_to_camera_joint: type fixed, parent camera_post_arm_link, child camera_link, origin xyz=0.02 0 0.027 rpy=0.0 0.2617993877991494 0.0
- added joint camera_post_to_camera_post_arm_joint: type fixed, parent camera_post_link, child camera_post_arm_link, origin xyz=0.03 0 0.08825000000000008 rpy=0 0 0
- added joint camera_to_camera_link_optical_joint: type fixed, parent camera_link, child camera_link_optical, origin xyz=0 0 0 rpy=-1.5707963267948966 0 -1.5707963267948966
- added joint chasis_cpu_cases_joint: type fixed, parent base_link, child cpu_cases_link, origin xyz=-0.15 0 1.53 rpy=0 0 0
- added joint front_left_chassis_engine_joint: type revolute, parent base_link, child front_left_engine_link, origin xyz=1.1 1 0 rpy=0.0 0.0 0, axis 0 0 1, limit lower=-3.141592653589793 upper=3.141592653589793 effort=10 velocity=10
- added joint front_left_engine_propeller_joint: type continuous, parent front_left_engine_link, child front_left_propeller_link, origin xyz=-0.278156 0 -0.509371 rpy=0 0 0, axis 1 0 0, limit effort=100 velocity=100
- added joint front_right_chassis_engine_joint: type revolute, parent base_link, child front_right_engine_link, origin xyz=1.1 -1 0 rpy=0.0 0.0 0, axis 0 0 1, limit lower=-3.141592653589793 upper=3.141592653589793 effort=10 velocity=10
- added joint front_right_engine_propeller_joint: type continuous, parent front_right_engine_link, child front_right_propeller_link, origin xyz=-0.278156 0 -0.509371 rpy=0 0 0, axis 1 0 0, limit effort=100 velocity=100
- added joint gps_wamv_joint: type revolute, parent base_link, child gps_wamv_link, origin xyz=-0.85 0.0 1.3 rpy=0.0 0.0 0.0, axis 0 0 1, limit lower=0.0 upper=0 effort=1000.0 velocity=0
- added joint imu_wamv_joint: type revolute, parent base_link, child imu_wamv_link, origin xyz=0.3 -0.2 1.3 rpy=0.0 0.0 0.0, axis 0 0 1, limit lower=0.0 upper=0 effort=1000.0 velocity=0
- added joint left_chasis_battery_joint: type fixed, parent base_link, child left_battery_link, origin xyz=0 1 0.45 rpy=0 0 0
- added joint lidar_wamv_post_arm_to_lidar_wamv_joint: type fixed, parent lidar_wamv_post_arm_link, child lidar_wamv_link, origin xyz=0.04 0 0.05 rpy=0.0 0.13962634015954636 0.0
- added joint lidar_wamv_post_to_lidar_wamv_post_arm_joint: type fixed, parent lidar_wamv_post_link, child lidar_wamv_post_arm_link, origin xyz=0.03 0 0.22675000000000006 rpy=0 0 0
- added joint receiver_pinger_joint: type revolute, parent base_link, child receiver, origin xyz=0 0 0 rpy=0 0 0, axis 0 0 1, limit lower=0.0 upper=0 effort=1000.0 velocity=0
- added joint right_chasis_battery_joint: type fixed, parent base_link, child right_battery_link, origin xyz=0 -1 0.45 rpy=0 0 0

File: seaweed_description/urdf/x_drive_wamv/wamv_target.urdf (robot description, URDF)
Before this commit: robot WAM-V, 24 links, 23 joints
Links:
- removed link wamv/back_left_engine_link
- removed link wamv/back_left_propeller_link
- removed link wamv/back_right_engine_link
- removed link wamv/back_right_propeller_link
- removed link wamv/ball_shooter_base_link
- removed link wamv/ball_shooter_launcher_link
- removed link wamv/base_link
- removed link wamv/camera_link
- removed link wamv/camera_link_optical
- removed link wamv/camera_post_arm_link
- removed link wamv/camera_post_link
- removed link wamv/cpu_cases_link
- removed link wamv/front_left_engine_link
- removed link wamv/front_left_propeller_link
- removed link wamv/front_right_engine_link
- removed link wamv/front_right_propeller_link
- removed link wamv/gps_wamv_link
- removed link wamv/imu_wamv_link
- removed link wamv/left_battery_link
- removed link wamv/lidar_wamv_link
- removed link wamv/lidar_wamv_post_arm_link
- removed link wamv/lidar_wamv_post_link
- removed link wamv/receiver
- removed link wamv/right_battery_link
- added link back_left_engine_link, mass 15; collision box size=0.12 0.15 0.12; collision box size=0.2 0.15 0.83
- added link back_left_propeller_link, mass 0.5; collision cylinder length=0.18 radius=0.24; visual mesh filename=package://wamv_description/models/propeller/mesh/propeller.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
- added link back_right_engine_link, mass 15; collision box size=0.12 0.15 0.12; collision box size=0.2 0.15 0.83
- added link back_right_propeller_link, mass 0.5; collision cylinder length=0.18 radius=0.24; visual mesh filename=package://wamv_description/models/propeller/mesh/propeller.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
- added link ball_shooter_base_link, mass 0.5; visual mesh filename=package://vrx_gazebo/models/ball_shooter/meshes/ball_shoote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
- added link ball_shooter_launcher_link, mass 0.5; collision box size=0.3 0.3 0.2; visual mesh filename=package://vrx_gazebo/models/ball_shooter/meshes/ball_shoote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
- added link base_link, mass 180.0; collision box size=0.65 0.2 0.1; collision box size=0.65 0.2 0.1
- added link camera_link, mass 0.3; collision box size=0.036 0.03 0.03; collision cylinder length=0.042 radius=0.015
- added link camera_link_optical
- added link camera_post_arm_link, mass 0.1; collision cylinder length=0.065 radius=0.008; visual mesh filename=package://vrx_gazebo/models/sensor_post/mesh/sensor_post_ar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
- added link camera_post_link, mass 0.15885000000000002; collision cylinder length=0.17650000000000002 radius=0.0076; visual cylinder length=0.17650000000000002 radius=0.0076
- added link cpu_cases_link, mass 20; collision box size=0.375 0.64 0.28; collision box size=0.595 0.83 0.47
- added link front_left_engine_link, mass 15; collision box size=0.12 0.15 0.12; collision box size=0.2 0.15 0.83
- added link front_left_propeller_link, mass 0.5; collision cylinder length=0.18 radius=0.24; visual mesh filename=package://wamv_description/models/propeller/mesh/propeller.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
- added link front_right_engine_link, mass 15; collision box size=0.12 0.15 0.12; collision box size=0.2 0.15 0.83
- added link front_right_propeller_link, mass 0.5; collision cylinder length=0.18 radius=0.24; visual mesh filename=package://wamv_description/models/propeller/mesh/propeller.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
- added link gps_wamv_link, mass 1; collision cylinder length=0.05 radius=0.015; collision cylinder length=0.1 radius=0.15
- added link imu_wamv_link, mass 0.1; collision box size=0.05 0.025 0.005; visual box size=0.05 0.025 0.005
- added link left_battery_link, mass 23.5; collision box size=.6 .4 .31; visual mesh filename=package://vrx_gazebo/models/battery/mesh/battery.dae
- added link lidar_wamv_link, mass 1; collision cylinder length=0.075 radius=0.055; visual mesh filename=package://vrx_gazebo/models/3d_lidar/mesh/3d_lidar.dae
- added link lidar_wamv_post_arm_link, mass 0.1; collision cylinder length=0.065 radius=0.008; visual mesh filename=package://vrx_gazebo/models/sensor_post/mesh/sensor_post_ar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
- added link lidar_wamv_post_link, mass 0.40815000000000007; collision cylinder length=0.45350000000000007 radius=0.0076; visual cylinder length=0.45350000000000007 radius=0.0076
- added link receiver, mass 0.1; visual sphere radius=0.01
- added link right_battery_link, mass 23.5; collision box size=.6 .4 .31; visual mesh filename=package://vrx_gazebo/models/battery/mesh/battery.dae
Joints:
- removed joint wamv/back_left_chassis_engine_joint
- removed joint wamv/back_left_engine_propeller_joint
- removed joint wamv/back_right_chassis_engine_joint
- removed joint wamv/back_right_engine_propeller_joint
- removed joint wamv/ball_shooter_base_joint
- removed joint wamv/ball_shooter_launcher_joint
- removed joint wamv/base_to_camera_post_joint
- removed joint wamv/base_to_lidar_wamv_post_joint
- removed joint wamv/camera_post_arm_to_camera_joint
- removed joint wamv/camera_post_to_camera_post_arm_joint
- removed joint wamv/camera_to_camera_link_optical_joint
- removed joint wamv/chasis_cpu_cases_joint
- removed joint wamv/front_left_chassis_engine_joint
- removed joint wamv/front_left_engine_propeller_joint
- removed joint wamv/front_right_chassis_engine_joint
- removed joint wamv/front_right_engine_propeller_joint
- removed joint wamv/gps_wamv_joint
- removed joint wamv/imu_wamv_joint
- removed joint wamv/left_chasis_battery_joint
- removed joint wamv/lidar_wamv_post_arm_to_lidar_wamv_joint
- removed joint wamv/lidar_wamv_post_to_lidar_wamv_post_arm_joint
- removed joint wamv/receiver_pinger_joint
- removed joint wamv/right_chasis_battery_joint
- added joint back_left_chassis_engine_joint: type revolute, parent base_link, child back_left_engine_link, origin xyz=-2.4 1 0 rpy=0.0 0.0 0.7854, axis 0 0 1, limit lower=-3.141592653589793 upper=3.141592653589793 effort=10 velocity=10
- added joint back_left_engine_propeller_joint: type continuous, parent back_left_engine_link, child back_left_propeller_link, origin xyz=-0.278156 0 -0.509371 rpy=0 0 0, axis 1 0 0, limit effort=100 velocity=100
- added joint back_right_chassis_engine_joint: type revolute, parent base_link, child back_right_engine_link, origin xyz=-2.4 -1 0 rpy=0.0 0.0 -0.7854, axis 0 0 1, limit lower=-3.141592653589793 upper=3.141592653589793 effort=10 velocity=10
- added joint back_right_engine_propeller_joint: type continuous, parent back_right_engine_link, child back_right_propeller_link, origin xyz=-0.278156 0 -0.509371 rpy=0 0 0, axis 1 0 0, limit effort=100 velocity=100
- added joint ball_shooter_base_joint: type revolute, parent base_link, child ball_shooter_base_link, origin xyz=0.55 -0.3 1.3 rpy=0 0 0.0, axis 0 0 1, limit lower=0.0 upper=0 effort=1000.0 velocity=0
- added joint ball_shooter_launcher_joint: type revolute, parent ball_shooter_base_link, child ball_shooter_launcher_link, origin xyz=-0.0204 0 0.107877 rpy=0 -0.3490658503988659 0, axis 0 0 1, limit lower=0.0 upper=0 effort=1000.0 velocity=0
- added joint base_to_camera_post_joint: type fixed, parent base_link, child camera_post_link, origin xyz=0.7 0.0 1.38475 rpy=0 0 0.0
- added joint base_to_lidar_wamv_post_joint: type fixed, parent base_link, child lidar_wamv_post_link, origin xyz=0.6299999999999999 0.0 1.52325 rpy=0 0 0.0
- added joint camera_post_arm_to_camera_joint: type fixed, parent camera_post_arm_link, child camera_link, origin xyz=0.02 0 0.027 rpy=0.0 0.2617993877991494 0.0
- added joint camera_post_to_camera_post_arm_joint: type fixed, parent camera_post_link, child camera_post_arm_link, origin xyz=0.03 0 0.08825000000000008 rpy=0 0 0
- added joint camera_to_camera_link_optical_joint: type fixed, parent camera_link, child camera_link_optical, origin xyz=0 0 0 rpy=-1.5707963267948966 0 -1.5707963267948966
- added joint chasis_cpu_cases_joint: type fixed, parent base_link, child cpu_cases_link, origin xyz=-0.15 0 1.53 rpy=0 0 0
- added joint front_left_chassis_engine_joint: type revolute, parent base_link, child front_left_engine_link, origin xyz=1.1 1 0 rpy=0.0 0.0 -0.7854, axis 0 0 1, limit lower=-3.141592653589793 upper=3.141592653589793 effort=10 velocity=10
- added joint front_left_engine_propeller_joint: type continuous, parent front_left_engine_link, child front_left_propeller_link, origin xyz=-0.278156 0 -0.509371 rpy=0 0 0, axis 1 0 0, limit effort=100 velocity=100
- added joint front_right_chassis_engine_joint: type revolute, parent base_link, child front_right_engine_link, origin xyz=1.1 -1 0 rpy=0.0 0.0 0.7854, axis 0 0 1, limit lower=-3.141592653589793 upper=3.141592653589793 effort=10 velocity=10
- added joint front_right_engine_propeller_joint: type continuous, parent front_right_engine_link, child front_right_propeller_link, origin xyz=-0.278156 0 -0.509371 rpy=0 0 0, axis 1 0 0, limit effort=100 velocity=100
- added joint gps_wamv_joint: type revolute, parent base_link, child gps_wamv_link, origin xyz=-0.85 0.0 1.3 rpy=0.0 0.0 0.0, axis 0 0 1, limit lower=0.0 upper=0 effort=1000.0 velocity=0
- added joint imu_wamv_joint: type revolute, parent base_link, child imu_wamv_link, origin xyz=0.3 -0.2 1.3 rpy=0.0 0.0 0.0, axis 0 0 1, limit lower=0.0 upper=0 effort=1000.0 velocity=0
- added joint left_chasis_battery_joint: type fixed, parent base_link, child left_battery_link, origin xyz=0 1 0.45 rpy=0 0 0
- added joint lidar_wamv_post_arm_to_lidar_wamv_joint: type fixed, parent lidar_wamv_post_arm_link, child lidar_wamv_link, origin xyz=0.04 0 0.05 rpy=0.0 0.13962634015954636 0.0
- added joint lidar_wamv_post_to_lidar_wamv_post_arm_joint: type fixed, parent lidar_wamv_post_link, child lidar_wamv_post_arm_link, origin xyz=0.03 0 0.22675000000000006 rpy=0 0 0
- added joint receiver_pinger_joint: type revolute, parent base_link, child receiver, origin xyz=0 0 0 rpy=0 0 0, axis 0 0 1, limit lower=0.0 upper=0 effort=1000.0 velocity=0
- added joint right_chasis_battery_joint: type fixed, parent base_link, child right_battery_link, origin xyz=0 -1 0.45 rpy=0 0 0

Commit message: fix: misc fixes during migration, updated perception util methods, added get_robot_pose helper

File: seaweed_description/urdf/diff_thrust_wamv/wamv_target.urdf (robot description, URDF)
Before this commit: robot WAM-V, 24 links, 23 joints
Links:
- link cpu_cases_link: geometry collision box size=0.375 0.64 0.28; collision box size=0.595 0.83 0.47
